Commit message: second try change urdf

File: python/assets/robot_properties_fingers/urdf/trifinger_edu.urdf (robot description, URDF)
Before this commit: robot trifingeredu, 17 links, 16 joints
Links:
- link trifinger_base_link: mass None -> 0

Commit message: the new urdf is working fine, tests are passing

File: python/assets/robot_properties_fingers/urdf/trifinger_edu.urdf (robot description, URDF)
Before this commit: robot trifingeredu, 17 links, 16 joints
Links:
- link finger_base_link_0: geometry visual mesh filename=package://robot_properties_fingers/meshes/stl/edu/base_back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 scale=1 1 1; visual mesh filename=package://robot_properties_fingers/meshes/stl/edu/base_fron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 scale=1 1 1
- link finger_base_link_120: geometry visual mesh filename=package://robot_properties_fingers/meshes/stl/edu/base_back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 scale=1 1 1; visual mesh filename=package://robot_properties_fingers/meshes/stl/edu/base_fron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 scale=1 1 1
- link finger_base_link_240: geometry visual mesh filename=package://robot_properties_fingers/meshes/stl/edu/base_back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 scale=1 1 1; visual mesh filename=package://robot_properties_fingers/meshes/stl/edu/base_fron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 scale=1 1 1
